File: hardware/C23/BSN-C23.kicad_sch (KiCad schematic)
At the start: 45 parts, among them J1 Conn_Coaxial_Small, U1 nRF54L05-QFXX, U2 SHTC3, U3 HDC2010, U4 CC2340R52E0RGER, X1 32MHz, X2 32.768kHz

Commit message: Cleaned up libraries for both variants
Renamed the project libraries to BSN-N54 / BSN-C23 and updated lib tables and all references, removed Nordic parts and the unused 40-pin CC2340 package from the C23 library, synced Antenna symbol fields to N54, updated READMEs.
Parts:
- AE1: footprint BLE_Sensor_Node:AANI-CH-0138-Q-T -> BSN-C23:AANI-CH-0138-Q-T; symbol BLE_Sensor_Node:Antenna -> BSN-C23:Antenna
- U1: footprint BLE_Sensor_Node:VQFN-48-1EP_6x6mm_P0.4mm_EP4.1x4.1mm_ThermalVias -> BSN-C23:VQFN-48-1EP_6x6mm_P0.4mm_EP4.1x4.1mm_ThermalVias; symbol BLE_Sensor_Node:nRF54L05-QFXX -> BSN-C23:nRF54L05-QFXX
- U3: footprint BLE_Sensor_Node:HDC2010 -> BSN-C23:HDC2010; symbol BLE_Sensor_Node:HDC2010Y -> BSN-C23:HDC2010Y
- U4: footprint BLE_Sensor_Node:Texas_RGE0024B_VQFN-24-1EP_4x4mm_P0.5mm_EP2.45x2.45mm_ThermalVias -> BSN-C23:Texas_RGE0024B_VQFN-24-1EP_4x4mm_P0.5mm_EP2.45x2.45mm_ThermalVias; symbol BLE_Sensor_Node:CC2340R52E0RGER -> BSN-C23:CC2340R52E0RGER
Changed lines of the file:
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@@
 	)
 	(symbol
-		(lib_id "BLE_Sensor_Node:HDC2010Y")
+		(lib_id "BSN-C23:HDC2010Y")
 		(at 67.31 226.06 0)
 		(unit 1)
@@
 			)
 		)
-		(property "Footprint" "BLE_Sensor_Node:HDC2010"
+		(property "Footprint" "BSN-C23:HDC2010"
 			(at 67.31 226.06 0)
 			(hide yes)
@@
 	)
 	(symbol
-		(lib_id "BLE_Sensor_Node:CC2340R52E0RGER")
+		(lib_id "BSN-C23:CC2340R52E0RGER")
 		(at 140.97 168.91 0)
 		(unit 1)
@@
 			)
 		)
-		(property "Footprint" "BLE_Sensor_Node:Texas_RGE0024B_VQFN-24-1EP_4x4mm_P0.5mm_EP2.45x2.45mm_ThermalVias"
+		(property "Footprint" "BSN-C23:Texas_RGE0024B_VQFN-24-1EP_4x4mm_P0.5mm_EP2.45x2.45mm_ThermalVias"
 			(at 140.97 168.91 0)
 			(hide yes)
@@
 	)
 	(symbol
-		(lib_id "BLE_Sensor_Node:nRF54L05-QFXX")
+		(lib_id "BSN-C23:nRF54L05-QFXX")
 		(at 207.01 147.32 0)
 		(unit 1)
@@
 			)
 		)
-		(property "Footprint" "BLE_Sensor_Node:VQFN-48-1EP_6x6mm_P0.4mm_EP4.1x4.1mm_ThermalVias"
+		(property "Footprint" "BSN-C23:VQFN-48-1EP_6x6mm_P0.4mm_EP4.1x4.1mm_ThermalVias"
 			(at 207.01 220.98 0)
 			(hide yes)
@@
 	)
 	(symbol
-		(lib_id "BLE_Sensor_Node:Antenna")
+		(lib_id "BSN-C23:Antenna")
 		(at 312.42 142.24 0)
 		(unit 1)
@@
 			)
 		)
-		(property "Footprint" "BLE_Sensor_Node:AANI-CH-0138-Q-T"
+		(property "Footprint" "BSN-C23:AANI-CH-0138-Q-T"
 			(at 312.42 142.24 0)
 			(hide yes)

Commit message: C23 variant schematics and component allocation fixes - work in progress
Parts:
- removed C15: 2.0p, Capacitor_SMD:C_0402_1005Metric, symbol Device:C_Small
- removed C7: 2.2u, Capacitor_SMD:C_0402_1005Metric, symbol Device:C_Small
- removed FB1: 100R@100MHz, Inductor_SMD:L_0603_1608Metric, symbol Device:FerriteBead_Small
- removed L3, L4: 3.5n, Inductor_SMD:L_0402_1005Metric, symbol Device:L_Small
- removed R4: R, Resistor_SMD:R_0201_0603Metric, symbol Device:R
- removed U1: nRF54L05-QFXX, BSN-C23:VQFN-48-1EP_6x6mm_P0.4mm_EP4.1x4.1mm_ThermalVias, symbol BSN-C23:nRF54L05-QFXX
- added C11: 100n, Capacitor_SMD:C_0402_1005Metric, symbol Device:C_Small
- added C13: 1u, Capacitor_SMD:C_0603_1608Metric, symbol Device:C_Small
- added C14: C, Capacitor_SMD:C_0402_1005Metric, symbol Device:C_Small
- added C18: 1.5p, Capacitor_SMD:C_0402_1005Metric, symbol Device:C_Small
- added C19, C20: 15p, Capacitor_SMD:C_0402_1005Metric, symbol Device:C_Small
- added TP3, TP6: TestPoint, TestPoint:TestPoint_Pad_D1.0mm, symbol Connector:TestPoint
- C16: value 0.3p -> C; DigiKey 490-17132-1-ND -> (none); now not fitted; now left out of the parts list
- C17: renamed from C14; DigiKey 712-QLCD250Q1R5B1GV001TCT-ND -> 490-8087-1-ND
- C5: value 100n -> C; AX 27726 -> (none); now not fitted; now left out of the parts list
- C6: value 2.2u -> 10u; footprint Capacitor_SMD:C_0402_1005Metric -> Capacitor_SMD:C_0603_1608Metric; AX (none) -> 27204; DigiKey 490-12731-1-ND -> (none)
- C8: value 10n -> C; DigiKey 490-3194-1-ND -> (none); now not fitted; now left out of the parts list
- C9: value 10n -> 100n; AX (none) -> 27726; DigiKey 490-3194-1-ND -> (none)
- L1: value 4.7u -> 10u; DigiKey 490-12065-1-ND -> (none)
- L2: value 2.7n -> 2.8n; DigiKey 490-15398-1-ND -> 490-LQW15AN2N8G80DCT-ND
- R3: renamed from R1; value 1k -> 100k; AX 201001 -> (none)
- U1: renamed from U4; DigiKey (none) -> 296-CC2340R52E0RGERCT-ND
- X1: renamed from X2; now not fitted; now left out of the parts list
- X2: renamed from X1; value 32MHz -> 48MHz; DigiKey 478-CX3225FB32000C0FZZH1CT-ND -> ECS-480-8-33B-CWN-TR3
- renumbered C12 to C1, C4 to C10, C3 to C12, C2 to C15, C11 to C2, C10 to C3, C13 to C4, C1 to C7, L5 to L3, L6 to L4, L7 to L5, R2 to R1, R3 to R2, TP5 to TP1, TP4 to TP10, TP6 to TP2, TP2 to TP4, TP3 to TP5, TP8 to TP7, TP7 to TP8, TP1 to TP9
Connections:
- net XC1 is gone; now on net X48P: X2.1
- net XC2 is gone; now on net X48N: X2.3
- net XL1 is gone; now on net X32N: X1.2
- net XL2 is gone; now on net X32P: X1.1
- net GND: now also U1.23 (GND), U1.25 (GND), C11.2, C13.2, C14.2, C18.2
- net INT: now also U1.10 (DIO21_A10)
- net SCL: now also U1.12 (DIO24_A7)
- net SDA: now also U1.5 (DIO12)
- net VDD: now also R3.2, U1.11 (VDDS), U1.18 (VDDS), U1.24 (VDDS); no longer C5.1
- net ~{RESET}: now also C4.1, R3.1, U1.13 (RSTN); no longer R3.2
- net at C9.1: now also C6.1, L1.1, U1.2 (VDDR), U1.20 (VDDR), C11.1; no longer C8.1
- net at L3.2, L4.1: now also C20.1; no longer C16.1
- net at U1.1 (ANT): now also C17.1, L2.1
- net X32P: now reaches U1.14 (DIO3_X32P)
- net X32P: now also C8.1
- net X32N: now reaches U1.15 (DIO4_X32N)
- net X32N: now also C5.1
- net at U1.16 (VDDD): now also C13.1
- net at U1.17 (DCDC): now also L1.2
- net X48P: now reaches U1.21 (X48P)
- net X48P: now also C16.1
- net X48N: now reaches U1.22 (X48N)
- net X48N: now also C14.1
- net TXD: now reaches U1.6 (DIO13)
- net TXD: now also TP3.1
- net at U1.7 (DIO16_SWDIO): now also TP4.1
- net at U1.8 (DIO17_SWDCK): now also TP5.1
- net RXD: now reaches U1.9 (DIO20_A11)
- net RXD: now also TP6.1
- net at L2.2: now also C18.1, C19.1, C20.2; no longer C17.1
- net at J1.1 (In): now also C19.2
- no-connect marks 26 -> 3
Other:
- moved on the sheet: AE1, C10, C12, C15, C17, C4, C7, J1, L1, L2, L3, L4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

Commit message: Matched components & Footrpints. Small routing changes on N54
Parts:
- C13: footprint Capacitor_SMD:C_0603_1608Metric -> Capacitor_SMD:C_0402_1005Metric; AX (none) -> 27730
- C3: DigiKey 490-9969-1-ND -> 490-GRM21BR60J107ME15KCT-ND
- L1: footprint Inductor_SMD:L_0402_1005Metric -> Inductor_SMD:L_0603_1608Metric; AX (none) -> 73170
- R3: AX (none) -> 201003
- X2: DigiKey ECS-480-8-33B-CWN-TR3 -> 50-ECS-480-8-33B-CWN-TR3CT-ND
Changed lines of the file:
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@@
 			)
 		)
-		(property "AX" ""
+		(property "AX" "201003"
 			(at 133.35 223.52 0)
 			(hide yes)
@@
 			)
 		)
-		(property "DigiKey" "ECS-480-8-33B-CWN-TR3"
+		(property "DigiKey" "50-ECS-480-8-33B-CWN-TR3CT-ND"
 			(at 182.88 167.64 0)
 			(hide yes)
@@
 			)
 		)
-		(property "Footprint" "Capacitor_SMD:C_0603_1608Metric"
+		(property "Footprint" "Capacitor_SMD:C_0402_1005Metric"
 			(at 189.23 156.21 0)
 			(hide yes)
@@
 			)
 		)
-		(property "AX" ""
+		(property "AX" "27730"
 			(at 189.23 156.21 0)
 			(hide yes)
@@
 			)
 		)
-		(property "Footprint" "Inductor_SMD:L_0402_1005Metric"
+		(property "Footprint" "Inductor_SMD:L_0603_1608Metric"
 			(at 196.85 146.05 0)
 			(hide yes)
@@
 			)
 		)
-		(property "DigiKey" ""
+		(property "AX" "73170"
 			(at 196.85 146.05 0)
 			(hide yes)
@@
 			)
 		)
-		(property "DigiKey" "490-9969-1-ND"
+		(property "DigiKey" "490-GRM21BR60J107ME15KCT-ND"
 			(at 67.31 127 0)
 			(hide yes)

Commit message: Started C23 varant layout
Parts:
- renumbered C7 to C1, C6 to C10, C9 to C11, C11 to C12, C16 to C15, C2 to C16, C1 to C17, C4 to C18, C5 to C19, C10 to C2, C8 to C20, C12 to C3, C15 to C4, C3 to C5, C20 to C6, C17 to C7, C18 to C8, C19 to C9, L2 to L1, L4 to L2, L5 to L4, L1 to L5, TP2 to TP1, TP3 to TP2, TP4 to TP3, TP1 to TP4, X2 to X1, X1 to X2
Other:
- moved on the sheet: C10, C11, C12, L5
