File: hardware/N54/BSN-N54.kicad_sch (KiCad schematic)
At the start: 44 parts, among them J1 Conn_Coaxial_Small, U1 nRF54L05-QFXX, U2 SHTC3, U3 HDC2010, X1 32MHz, X2 32.768kHz

Commit message: Adopted BSN-<variant>-<rev> naming scheme
Renamed variant folders to N54/C23 and the nRF KiCad project to BSN-N54, documented the naming scheme in README.
Other:
- title: BLE Sensor Node (nRF54L variant) -> BSN-N54 - BLE Sensor Node, nRF54L variant

Commit message: Cleaned up libraries for both variants
Renamed the project libraries to BSN-N54 / BSN-C23 and updated lib tables and all references, removed Nordic parts and the unused 40-pin CC2340 package from the C23 library, synced Antenna symbol fields to N54, updated READMEs.
Parts:
- AE1: footprint BLE_Sensor_Node:AANI-CH-0138-Q-T -> BSN-N54:AANI-CH-0138-Q-T; symbol BLE_Sensor_Node:Antenna -> BSN-N54:Antenna
- U1: footprint BLE_Sensor_Node:VQFN-48-1EP_6x6mm_P0.4mm_EP4.1x4.1mm_ThermalVias -> BSN-N54:VQFN-48-1EP_6x6mm_P0.4mm_EP4.1x4.1mm_ThermalVias; symbol BLE_Sensor_Node:nRF54L05-QFXX -> BSN-N54:nRF54L05-QFXX
- U3: footprint BLE_Sensor_Node:HDC2010 -> BSN-N54:HDC2010; symbol BLE_Sensor_Node:HDC2010Y -> BSN-N54:HDC2010Y
Changed lines of the file:
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@@
 	)
 	(symbol
-		(lib_id "BLE_Sensor_Node:HDC2010Y")
+		(lib_id "BSN-N54:HDC2010Y")
 		(at 67.31 226.06 0)
 		(unit 1)
@@
 			)
 		)
-		(property "Footprint" "BLE_Sensor_Node:HDC2010"
+		(property "Footprint" "BSN-N54:HDC2010"
 			(at 67.31 226.06 0)
 			(hide yes)
@@
 	)
 	(symbol
-		(lib_id "BLE_Sensor_Node:nRF54L05-QFXX")
+		(lib_id "BSN-N54:nRF54L05-QFXX")
 		(at 207.01 147.32 0)
 		(unit 1)
@@
 			)
 		)
-		(property "Footprint" "BLE_Sensor_Node:VQFN-48-1EP_6x6mm_P0.4mm_EP4.1x4.1mm_ThermalVias"
+		(property "Footprint" "BSN-N54:VQFN-48-1EP_6x6mm_P0.4mm_EP4.1x4.1mm_ThermalVias"
 			(at 207.01 220.98 0)
 			(hide yes)
@@
 	)
 	(symbol
-		(lib_id "BLE_Sensor_Node:Antenna")
+		(lib_id "BSN-N54:Antenna")
 		(at 312.42 142.24 0)
 		(unit 1)
@@
 			)
 		)
-		(property "Footprint" "BLE_Sensor_Node:AANI-CH-0138-Q-T"
+		(property "Footprint" "BSN-N54:AANI-CH-0138-Q-T"
 			(at 312.42 142.24 0)
 			(hide yes)

Commit message: C23 variant schematics and component allocation fixes - work in progress
Parts:
- C14: DigiKey 712-QLCD250Q1R5B1GV001TCT-ND -> 490-8087-1-ND
Changed lines of the file:
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@@
 			)
 		)
-		(property "DigiKey" "712-QLCD250Q1R5B1GV001TCT-ND"
+		(property "DigiKey" "490-8087-1-ND"
 			(at 247.65 149.86 0)
 			(hide yes)

Commit message: Matched components & Footrpints. Small routing changes on N54
Parts:
- C10: DigiKey 490-9969-1-ND -> 490-GRM21BR60J107ME15KCT-ND
- C16: DigiKey 490-17132-1-ND -> 490-11248-1-ND
- C6, C7: DigiKey 490-12731-1-ND -> 445-9028-1-ND
- C8, C9: DigiKey 490-3194-1-ND -> 490-4516-1-ND
- L1: footprint Inductor_SMD:L_0402_1005Metric -> Inductor_SMD:L_0603_1608Metric
Changed lines of the file:
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@@
 			)
 		)
-		(property "DigiKey" "490-12731-1-ND"
+		(property "DigiKey" "445-9028-1-ND"
 			(at 265.43 99.06 0)
 			(hide yes)
@@
 			)
 		)
-		(property "DigiKey" "490-12731-1-ND"
+		(property "DigiKey" "445-9028-1-ND"
 			(at 246.38 104.14 0)
 			(hide yes)
@@
 			)
 		)
-		(property "DigiKey" "490-17132-1-ND"
+		(property "DigiKey" "490-11248-1-ND"
 			(at 267.97 149.86 0)
 			(hide yes)
@@
 			)
 		)
-		(property "DigiKey" "490-3194-1-ND"
+		(property "DigiKey" "490-4516-1-ND"
 			(at 276.86 99.06 0)
 			(hide yes)
@@
 			)
 		)
-		(property "Footprint" "Inductor_SMD:L_0402_1005Metric"
+		(property "Footprint" "Inductor_SMD:L_0603_1608Metric"
 			(at 237.49 104.14 0)
 			(hide yes)
@@
 			)
 		)
-		(property "DigiKey" "490-3194-1-ND"
+		(property "DigiKey" "490-4516-1-ND"
 			(at 288.29 99.06 0)
 			(hide yes)
@@
 			)
 		)
-		(property "DigiKey" "490-9969-1-ND"
+		(property "DigiKey" "490-GRM21BR60J107ME15KCT-ND"
 			(at 67.31 127 0)
 			(hide yes)

Commit message: Added UART test points
Parts:
- added TP10, TP9: TestPoint, TestPoint:TestPoint_Pad_D1.0mm, symbol Connector:TestPoint
Connections:
- net TXD: now reaches U1.7 (P1.06)
- net TXD: now also TP9.1
- net RXD: now reaches U1.8 (P1.07)
- net RXD: now also TP10.1
- no-connect marks 26 -> 24
Changed lines of the file:
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@@
 	)
 	(no_connect
-		(at 179.07 149.86)
-	)
-	(no_connect
 		(at 179.07 152.4)
 	)
@@
 	)
 	(no_connect
-		(at 179.07 147.32)
-	)
-	(no_connect
 		(at 179.07 162.56)
 	)
@@
 	(wire
 		(pts
+			(xy 172.72 147.32) (xy 179.07 147.32)
+		)
+		(stroke
+			(width 0)
+			(type default)
+		)
+	)
+	(wire
+		(pts
 			(xy 207.01 207.01) (xy 207.01 205.74)
 		)
@@
 	(wire
 		(pts
+			(xy 172.72 149.86) (xy 179.07 149.86)
+		)
+		(stroke
+			(width 0)
+			(type default)
+		)
+	)
+	(wire
+		(pts
 			(xy 302.26 147.32) (xy 312.42 147.32)
 		)
@@
 		)
 	)
+	(label "RXD"
+		(at 172.72 149.86 0)
+		(effects
+			(font
+				(size 1.27 1.27)
+			)
+			(justify left bottom)
+		)
+	)
 	(label "SCL"
 		(at 167.64 129.54 0)
@@
 		)
 	)
+	(label "TXD"
+		(at 172.72 147.32 0)
+		(effects
+			(font
+				(size 1.27 1.27)
+			)
+			(justify left bottom)
+		)
+	)
 	(label "XC1"
 		(at 172.72 96.52 0)
@@
 	)
 	(symbol
+		(lib_id "Connector:TestPoint")
+		(at 172.72 149.86 90)
+		(unit 1)
+		(body_style 1)
+		(exclude_from_sim no)
+		(in_bom no)
+		(on_board yes)
+		(in_pos_files yes)
+		(dnp no)
+		(property "Reference" "TP10"
+			(at 168.148 149.86 90)
+			(show_name no)
+			(do_not_autoplace no)
+			(effects
+				(font
+					(size 1.27 1.27)
+				)
+				(justify left)
+			)
+		)
+		(property "Value" "TestPoint"
+			(at 167.64 148.5901 90)
+			(hide yes)
+			(show_name no)
+			(do_not_autoplace no)
+			(effects
+				(font
+					(size 1.27 1.27)
+				)
+				(justify left)
+			)
+		)
+		(property "Footprint" "TestPoint:TestPoint_Pad_D1.0mm"
+			(at 172.72 144.78 0)
+			(hide yes)
+			(show_name no)
+			(do_not_autoplace no)
+			(effects
+				(font
+					(size 1.27 1.27)
+				)
+			)
+		)
+		(property "Datasheet" ""
+			(at 172.72 144.78 0)
+			(hide yes)
+			(show_name no)
+			(do_not_autoplace no)
+			(effects
+				(font
+					(size 1.27 1.27)
+				)
+			)
+		)
+		(property "Description" "test point"
+			(at 172.72 149.86 0)
+			(hide yes)
+			(show_name no)
+			(do_not_autoplace no)
+			(effects
+				(font
+					(size 1.27 1.27)
+				)
+			)
+		)
+		(pin "1"
+		)
+		(instances
+			(project "BSN-N54"
+				(path "/3be841bb-f0fa-4f59-8a52-40b0b50ca4ae"
+					(reference "TP10")
+					(unit 1)
+				)
+			)
+		)
+	)
+	(symbol
 		(lib_id "power:VDD")
 		(at 97.79 201.93 0)
@@
 					(unit 1)
 				)
+			)
+		)
+	)
+	(symbol
+		(lib_id "Connector:TestPoint")
+		(at 172.72 147.32 90)
+		(unit 1)
+		(body_style 1)
+		(exclude_from_sim no)
+		(in_bom no)
+		(on_board yes)
+		(in_pos_files yes)
+		(dnp no)
+		(property "Reference" "TP9"
+			(at 168.148 147.32 90)
+			(show_name no)
+			(do_not_autoplace no)
+			(effects
+				(font
+					(size 1.27 1.27)
+				)
+				(justify left)
+			)
+		)
+		(property "Value" "TestPoint"
+			(at 167.64 146.0501 90)
+			(hide yes)
+			(show_name no)
+			(do_not_autoplace no)
+			(effects
+				(font
+					(size 1.27 1.27)
+				)
+				(justify left)
+			)
+		)
+		(property "Footprint" "TestPoint:TestPoint_Pad_D1.0mm"
+			(at 172.72 142.24 0)
+			(hide yes)
+			(show_name no)
+			(do_not_autoplace no)
+			(effects
+				(font
+					(size 1.27 1.27)
+				)
+			)
+		)
+		(property "Datasheet" ""
+			(at 172.72 142.24 0)
+			(hide yes)
+			(show_name no)
+			(do_not_autoplace no)
+			(effects
+				(font
+					(size 1.27 1.27)
+				)
+			)
+		)
+		(property "Description" "test point"
+			(at 172.72 147.32 0)
+			(hide yes)
+			(show_name no)
+			(do_not_autoplace no)
+			(effects
+				(font
+					(size 1.27 1.27)
+				)
+			)
+		)
+		(pin "1"
+		)
+		(instances
+			(project "BSN-N54"
+				(path "/3be841bb-f0fa-4f59-8a52-40b0b50ca4ae"
+					(reference "TP9")
+					(unit 1)
+				)
