File: hardware/panel/BSN-panel.kicad_pcb (KiCad board)
At the start: 4 copper layers, 84 x 70 mm, 232 parts, among them J1 Conn_Coaxial_Small, U1 CC2340R52E0RGER, U1 nRF54L05-QFXX, U2 SHTC3, U3 HDC2010, X1 32MHz, X1 48MHz, X2 32.768kHz

Commit message: More small fixes & Created new panel
Routing:
- net Board_2-GND: track 33.9 -> 26.7 mm, vias 80 -> 78
- net Board_3-GND: track 33.9 -> 26.7 mm, vias 80 -> 78
- net Board_0-VDD: track 32.8 -> 28.4 mm
- net Board_1-VDD: track 32.8 -> 28.4 mm
- net Board_0-GND: track 25.0 -> 27.3 mm
- net Board_1-GND: track 25.0 -> 27.3 mm
- net Board_3-VDD: track 36.0 -> 35.3 mm
- net Board_2-VDD: track 36.0 -> 35.3 mm
- net Board_2-Net-(U1-SWDCLK): track 16.5 -> 17.2 mm
- net Board_3-Net-(U1-SWDCLK): track 16.5 -> 17.2 mm
